File: fileCartridge.kicad_sch (KiCad schematic)
At the start: 20 parts, among them U11 74AHCV17A, U12 74AHCV17A, U13 74LVCH8T245, U14 74LVCH8T245, U5 74LVC06A, U8 74LVC1G06, U9 74LVCH8T245, X1 EXPANSION_PORT_C64_EDGE

Commit message: Update component prices
Parts:
- C4: Pricing (EUR) 0,10 -> 0,09
- U11, U12: Pricing (EUR) 0,44 -> 0,42
- U13, U14, U9: Pricing (EUR) 1,35 -> 1,26
- U5: Pricing (EUR) 1,01 -> 0,86
- U8: Pricing (EUR) 0.34 -> 0.32
Changed lines of the file:
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@@
       (effects (font (size 1.27 1.27)) hide)
     )
-    (property "Pricing (EUR)" "1,35" (at 44.45 69.85 0)
+    (property "Pricing (EUR)" "1,26" (at 44.45 69.85 0)
       (effects (font (size 1.27 1.27)) hide)
     )
@@
       (effects (font (size 1.27 1.27)) hide)
     )
-    (property "Pricing (EUR)" "1,35" (at 194.31 74.93 0)
+    (property "Pricing (EUR)" "1,26" (at 194.31 74.93 0)
       (effects (font (size 1.27 1.27)) hide)
     )
@@
       (effects (font (size 1.27 1.27)) hide)
     )
-    (property "Pricing (EUR)" "1,35" (at 142.24 74.93 0)
+    (property "Pricing (EUR)" "1,26" (at 142.24 74.93 0)
       (effects (font (size 1.27 1.27)) hide)
     )
@@
       (effects (font (size 1.27 1.27)) hide)
     )
-    (property "Pricing (EUR)" "0.34" (at 42.545 152.4 0)
+    (property "Pricing (EUR)" "0.32" (at 42.545 152.4 0)
       (effects (font (size 1.27 1.27)) hide)
     )
@@
       (effects (font (size 1.27 1.27)) hide)
     )
-    (property "Pricing (EUR)" "0,44" (at 173.99 125.73 0)
+    (property "Pricing (EUR)" "0,42" (at 173.99 125.73 0)
       (effects (font (size 1.27 1.27)) hide)
     )
@@
       (effects (font (size 1.27 1.27)) hide)
     )
-    (property "Pricing (EUR)" "0,44" (at 114.3 143.51 0)
+    (property "Pricing (EUR)" "0,42" (at 114.3 143.51 0)
       (effects (font (size 1.27 1.27)) hide)
     )
@@
       (effects (font (size 1.27 1.27)) hide)
     )
-    (property "Pricing (EUR)" "0,44" (at 128.27 34.29 0)
+    (property "Pricing (EUR)" "0,42" (at 128.27 34.29 0)
       (effects (font (size 1.27 1.27)) hide)
     )
@@
       (effects (font (size 1.27 1.27)) hide)
     )
-    (property "Pricing (EUR)" "0,44" (at 173.99 105.41 0)
+    (property "Pricing (EUR)" "0,42" (at 173.99 105.41 0)
       (effects (font (size 1.27 1.27)) hide)
     )
@@
       (effects (font (size 1.27 1.27)) hide)
     )
-    (property "Pricing (EUR)" "0,44" (at 165.1 114.3 0)
+    (property "Pricing (EUR)" "0,42" (at 165.1 114.3 0)
       (effects (font (size 1.27 1.27)) hide)
     )
@@
       (effects (font (size 1.27 1.27)) hide)
     )
-    (property "Pricing (EUR)" "1,01" (at 32.385 142.24 0)
+    (property "Pricing (EUR)" "0,86" (at 32.385 142.24 0)
       (effects (font (size 1.27 1.27)) hide)
     )
@@
       (effects (font (size 1.27 1.27)) hide)
     )
-    (property "Pricing (EUR)" "1,01" (at 20.955 152.4 0)
+    (property "Pricing (EUR)" "0,86" (at 20.955 152.4 0)
       (effects (font (size 1.27 1.27)) hide)
     )
@@
       (effects (font (size 1.27 1.27)) hide)
     )
-    (property "Pricing (EUR)" "1,01" (at 166.37 134.62 0)
+    (property "Pricing (EUR)" "0,86" (at 166.37 134.62 0)
       (effects (font (size 1.27 1.27)) hide)
     )
@@
       (effects (font (size 1.27 1.27)) hide)
     )
-    (property "Pricing (EUR)" "1,01" (at 80.01 142.24 0)
+    (property "Pricing (EUR)" "0,86" (at 80.01 142.24 0)
       (effects (font (size 1.27 1.27)) hide)
     )
@@
       (effects (font (size 1.27 1.27)) hide)
     )
-    (property "Pricing (EUR)" "1,01" (at 69.85 151.13 0)
+    (property "Pricing (EUR)" "0,86" (at 69.85 151.13 0)
       (effects (font (size 1.27 1.27)) hide)
     )
@@
       (effects (font (size 1.27 1.27)) hide)
     )
-    (property "Pricing (EUR)" "1,01" (at 105.41 34.29 0)
+    (property "Pricing (EUR)" "0,86" (at 105.41 34.29 0)
       (effects (font (size 1.27 1.27)) hide)
     )
@@
       (effects (font (size 1.27 1.27)) hide)
     )
-    (property "Pricing (EUR)" "0,10" (at 251.46 104.14 0)
+    (property "Pricing (EUR)" "0,09" (at 251.46 104.14 0)
       (effects (font (size 1.27 1.27)) hide)
     )
@@
       (effects (font (size 1.27 1.27)) hide)
     )
-    (property "Pricing (EUR)" "0,44" (at 140.97 153.67 0)
+    (property "Pricing (EUR)" "0,42" (at 140.97 153.67 0)
       (effects (font (size 1.27 1.27)) hide)
     )
@@
       (effects (font (size 1.27 1.27)) hide)
     )
-    (property "Pricing (EUR)" "0,44" (at 123.19 153.67 0)
+    (property "Pricing (EUR)" "0,42" (at 123.19 153.67 0)
       (effects (font (size 1.27 1.27)) hide)
     )
@@
       (effects (font (size 1.27 1.27)) hide)
     )
-    (property "Pricing (EUR)" "0,44" (at 95.25 153.67 0)
+    (property "Pricing (EUR)" "0,42" (at 95.25 153.67 0)
       (effects (font (size 1.27 1.27)) hide)
     )
@@
       (effects (font (size 1.27 1.27)) hide)
     )
-    (property "Pricing (EUR)" "0,44" (at 53.975 143.51 0)
+    (property "Pricing (EUR)" "0,42" (at 53.975 143.51 0)
       (effects (font (size 1.27 1.27)) hide)
     )
@@
       (effects (font (size 1.27 1.27)) hide)
     )
-    (property "Pricing (EUR)" "0,44" (at 163.83 158.75 0)
+    (property "Pricing (EUR)" "0,42" (at 163.83 158.75 0)
       (effects (font (size 1.27 1.27)) hide)
     )
@@
       (effects (font (size 1.27 1.27)) hide)
     )
-    (property "Pricing (EUR)" "0,44" (at 61.595 153.67 0)
+    (property "Pricing (EUR)" "0,42" (at 61.595 153.67 0)
       (effects (font (size 1.27 1.27)) hide)
     )
@@
       (effects (font (size 1.27 1.27)) hide)
     )
-    (property "Pricing (EUR)" "0,44" (at 132.08 143.51 0)
-      (effects (font (size 1.27 1.27)) hide)
-    )
+    (property "Pricing (EUR)" "0,42" (at 132.08 143.51 0)
+      (effects (font (size 1.27 1.27)) hide)
+    )
