File: fileClockport.kicad_sch (KiCad schematic)
At the start: 2 parts, among them J1 Conn_02x11_Odd_Even

Commit message: Update Mouser prices
Parts:
- J1: Pricing (EUR) 3,43 -> 4,37
- RN1: Pricing (EUR) 0,09 -> 0,10
Changed lines of the file:
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@@
       (effects (font (size 1.27 1.27)) hide)
     )
-    (property "Pricing (EUR)" "3,43" (id 7) (at 114.3 77.47 0)
+    (property "Pricing (EUR)" "4,37" (id 7) (at 114.3 77.47 0)
       (effects (font (size 1.27 1.27)) hide)
     )
@@
       (effects (font (size 1.27 1.27)) hide)
     )
-    (property "Pricing (EUR)" "0,09" (id 7) (at 171.45 78.74 0)
+    (property "Pricing (EUR)" "0,10" (id 7) (at 171.45 78.74 0)
       (effects (font (size 1.27 1.27)) hide)
     )

Commit message: Update component prices
Parts:
- J1: Pricing (EUR) 4,37 -> 4,14
- RN1: Pricing (EUR) 0,10 -> 0,09
Changed lines of the file:
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@@
       (effects (font (size 1.27 1.27)) hide)
     )
-    (property "Pricing (EUR)" "4,37" (at 114.3 77.47 0)
+    (property "Pricing (EUR)" "4,14" (at 114.3 77.47 0)
       (effects (font (size 1.27 1.27)) hide)
     )
@@
       (effects (font (size 1.27 1.27)) hide)
     )
-    (property "Pricing (EUR)" "0,10" (at 171.45 78.74 0)
+    (property "Pricing (EUR)" "0,09" (at 171.45 78.74 0)
       (effects (font (size 1.27 1.27)) hide)
     )
