File: fileSDMMC.kicad_sch (KiCad schematic)
At the start: 6 parts, among them J4 Micro_SD_Card_Det

Commit message: Fix some checker complaints
Changed lines of the file:
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@@
     (pin "9")
   )
+  (symbol (lib_id "power:PWR_FLAG") (at 121.92 78.74 0) (unit 1)
+    (in_bom yes) (on_board yes)
+    (property "Reference" "#FLG0108" (id 0) (at 121.92 76.835 0)
+      (effects (font (size 1.27 1.27)) hide)
+    )
+    (property "Value" "PWR_FLAG" (id 1) (at 121.92 74.3458 0))
+    (property "Footprint" "" (id 2) (at 121.92 78.74 0)
+      (effects (font (size 1.27 1.27)) hide)
+    )
+    (property "Datasheet" "~" (id 3) (at 121.92 78.74 0)
+      (effects (font (size 1.27 1.27)) hide)
+    )
+    (pin "1")
+  )
 )

Commit message: Update Mouser prices
Parts:
- C29: Pricing (EUR) 0,15 -> 0,18
- C70: Pricing (EUR) 0,09 -> 0,02
- FB1: Pricing (EUR) 0,09 -> 0,12
- J4: Pricing (EUR) 2,25 -> 2,48
- R28: Pricing (EUR) 0,11 -> 0,10
- RN7: Pricing (EUR) 0,09 -> 0,10
Changed lines of the file:
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@@
       (effects (font (size 1.27 1.27)) hide)
     )
-    (property "Pricing (EUR)" "0,09" (id 7) (at 58.42 102.87 0)
+    (property "Pricing (EUR)" "0,10" (id 7) (at 58.42 102.87 0)
       (effects (font (size 1.27 1.27)) hide)
     )
@@
       (effects (font (size 1.27 1.27)) hide)
     )
-    (property "Pricing (EUR)" "0,11" (id 7) (at 66.04 102.87 0)
+    (property "Pricing (EUR)" "0,10" (id 7) (at 66.04 102.87 0)
       (effects (font (size 1.27 1.27)) hide)
     )
@@
       (effects (font (size 1.27 1.27)) hide)
     )
-    (property "Pricing (EUR)" "0,09" (id 7) (at 109.22 78.74 0)
+    (property "Pricing (EUR)" "0,12" (id 7) (at 109.22 78.74 0)
       (effects (font (size 1.27 1.27)) hide)
     )
@@
       (effects (font (size 1.27 1.27)) hide)
     )
-    (property "Pricing (EUR)" "0,09" (id 7) (at 116.84 85.09 0)
+    (property "Pricing (EUR)" "0,02" (id 7) (at 116.84 85.09 0)
       (effects (font (size 1.27 1.27)) hide)
     )
@@
       (effects (font (size 1.27 1.27)) hide)
     )
-    (property "Pricing (EUR)" "0,15" (id 7) (at 121.92 85.09 0)
+    (property "Pricing (EUR)" "0,18" (id 7) (at 121.92 85.09 0)
       (effects (font (size 1.27 1.27)) hide)
     )
@@
       (effects (font (size 1.27 1.27)) hide)
     )
-    (property "Pricing (EUR)" "2,25" (id 7) (at 181.61 99.06 0)
+    (property "Pricing (EUR)" "2,48" (id 7) (at 181.61 99.06 0)
       (effects (font (size 1.27 1.27)) hide)
     )

Commit message: Update component prices
Parts:
- C29: Pricing (EUR) 0,18 -> 0,14
- FB1: Pricing (EUR) 0,12 -> 0,09
- J4: Pricing (EUR) 2,48 -> 2,43
- R28, RN7: Pricing (EUR) 0,10 -> 0,09
Changed lines of the file:
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@@
       (effects (font (size 1.27 1.27)) hide)
     )
-    (property "Pricing (EUR)" "0,10" (at 58.42 102.87 0)
+    (property "Pricing (EUR)" "0,09" (at 58.42 102.87 0)
       (effects (font (size 1.27 1.27)) hide)
     )
@@
       (effects (font (size 1.27 1.27)) hide)
     )
-    (property "Pricing (EUR)" "0,10" (at 66.04 102.87 0)
+    (property "Pricing (EUR)" "0,09" (at 66.04 102.87 0)
       (effects (font (size 1.27 1.27)) hide)
     )
@@
       (effects (font (size 1.27 1.27)) hide)
     )
-    (property "Pricing (EUR)" "0,12" (at 109.22 78.74 0)
+    (property "Pricing (EUR)" "0,09" (at 109.22 78.74 0)
       (effects (font (size 1.27 1.27)) hide)
     )
@@
       (effects (font (size 1.27 1.27)) hide)
     )
-    (property "Pricing (EUR)" "0,18" (at 121.92 85.09 0)
+    (property "Pricing (EUR)" "0,14" (at 121.92 85.09 0)
       (effects (font (size 1.27 1.27)) hide)
     )
@@
       (effects (font (size 1.27 1.27)) hide)
     )
-    (property "Pricing (EUR)" "2,48" (at 181.61 99.06 0)
-      (effects (font (size 1.27 1.27)) hide)
-    )
+    (property "Pricing (EUR)" "2,43" (at 181.61 99.06 0)
+      (effects (font (size 1.27 1.27)) hide)
+    )
